Commit message: fix: unify odometry source and clean TF tree
- Use encoder_positions as single odometry source
- Fix TF chain (odom -> base_footprint)
- Remove joint_states-based ambiguity
- Improve SimpleController stability

File: src/yakizbot_description/urdf/yakizbot.urdf.xacro (robot description, xacro)
@@ -12,40 +12,32 @@
   <!-- ================= PARAMETERS ================= -->
   <!-- Base dimensions -->
-  <xacro:property name="base_length"   value="0.40"/>   <!-- Length of robot base (X direction) -->
-  <xacro:property name="base_width"    value="0.295"/>  <!-- Width of robot base (Y direction) -->
-  <xacro:property name="base_height"   value="0.20"/>   <!-- Height of robot base (Z direction) -->
+  <xacro:property name="base_length"   value="0.40"/>
+  <xacro:property name="base_width"    value="0.295"/>
+  <xacro:property name="base_height"   value="0.20"/>
   <!-- Wheel dimensions -->
-  <xacro:property name="wheel_radius"  value="0.0425"/> <!-- Wheel radius -->
-  <xacro:property name="wheel_width"   value="0.038"/>   <!-- Wheel thickness -->
+  <xacro:property name="wheel_radius"  value="0.0425"/>
+  <xacro:property name="wheel_width"   value="0.038"/>
   <!-- Robot geometry -->
-  <xacro:property name="track"         value="0.28"/>   <!-- Distance between left and right wheels -->
-  <xacro:property name="wheelbase"     value="0.15"/>   <!-- Distance between front and rear wheels -->
+  <xacro:property name="track"         value="0.28"/>
+  <xacro:property name="wheelbase"     value="0.15"/>
   <!-- ================= MATERIALS ================= -->
-  <!-- Colors used for visualization -->
-  <!-- ================= MATERIALS ================= -->
-  <!-- Blue -->
   <material name="blue">
     <color rgba="0 0 1 1"/>
   </material>
-    <!-- black -->
   <material name="black">
     <color rgba="0 0 0 1"/>
   </material>
-    <!-- silver -->
   <material name="silver">
     <color rgba="0.79 0.82 0.93 1"/>
   </material>
-    <!-- dark_grey -->
   <material name="dark_grey">
     <color rgba="0.3 0.3 0.3 1"/>
   </material>
-  <!-- ================= BASE FOOTPRINT ================= -->
-  <!-- Virtual frame projected on ground (used in navigation) -->
+  <!-- ================================================= -->
   <link name="base_footprint"/>
-  <!-- Main robot body -->
+  <!-- ================= BASE LINK ================= -->
   <link name="base_link">
     <visual>
       <geometry>
-        <!-- Rectangular chassis -->
         <box size="${base_length} ${base_width} ${base_height}"/>
       </geometry>
@@ -53,5 +45,4 @@
     </visual>
     <collision>
-      <!-- Same geometry used for collision detection -->
       <geometry>
         <box size="${base_length} ${base_width} ${base_height}"/>
@@ -59,28 +50,23 @@
     </collision>
     <inertial>
-      <!-- Center of mass slightly above bottom -->
       <origin xyz="0 0 0.04"/>
       <mass value="3.0"/>
-      <!-- Approximate inertia tensor -->
-      <inertia ixx="0.05" ixy="0.0" ixz="0.0"
-               iyy="0.05" iyz="0.0"
-               izz="0.08"/>
+      <inertia
+        ixx="0.05"
+        ixy="0.0"
+        ixz="0.0"
+        iyy="0.05"
+        iyz="0.0"
+        izz="0.08"/>
     </inertial>
   </link>
-  <!-- Fixed joint between footprint and base -->
+  <!-- ================= BASE JOINT ================= -->
   <joint name="base_joint" type="fixed">
     <parent link="base_footprint"/>
     <child link="base_link"/>
-    <!-- Lift base so wheels touch ground -->
+    <!-- Lift robot body above ground -->
     <origin xyz="0 0 ${wheel_radius}" rpy="0 0 0"/>
   </joint>
   <!-- ================= WHEEL MACRO ================= -->
-  <!--
-    Macro to generate a wheel.
-    Parameters:
-    - name   : wheel name
-    - x_sign : +1 front, -1 rear
-    - y_sign : +1 left,  -1 right
-  -->
   <xacro:macro name="wheel" params="name x_sign y_sign">
     <!-- Wheel link -->
@@ -88,8 +74,7 @@
       <visual>
         <geometry>
-          <!-- Cylindrical wheel -->
           <cylinder radius="${wheel_radius}" length="${wheel_width}"/>
         </geometry>
-        <!-- Rotate so it spins around Y-axis -->
+        <!-- Cylinder rotated so wheel looks correct -->
         <origin rpy="${pi/2} 0 0"/>
         <material name="blue"/>
@@ -103,27 +88,36 @@
       <inertial>
         <mass value="0.3"/>
-        <!-- Simplified inertia -->
-        <inertia ixx="0.001" ixy="0" ixz="0"
-                 iyy="0.001" iyz="0"
-                 izz="0.001"/>
+        <inertia
+          ixx="0.001"
+          ixy="0"
+          ixz="0"
+          iyy="0.001"
+          iyz="0"
+          izz="0.001"/>
       </inertial>
     </link>
-    <!-- Wheel joint (continuous rotation) -->
-    <joint name="${name}_wheel" type="continuous">
+    <!-- Wheel joint -->
+    <joint name="${name}_wheel_joint" type="continuous">
       <parent link="base_link"/>
       <child link="${name}_wheel"/>
-      <!-- Position of wheel relative to base -->
-      <origin xyz="${x_sign * wheelbase/2}
-                   ${y_sign * track/2}
-                   ${-base_height/2}"
-              rpy="0 0 0"/>
-      <!-- Rotation axis (wheel spins around Y-axis) -->
+      <!-- Wheel position -->
+      <origin
+        xyz="${x_sign * wheelbase/2}
+             ${y_sign * track/2}
+             ${-base_height/2}"
+        rpy="0 0 0"/>
+      <!-- ================================================= -->
+      <!-- FIX: wheel rotation axis -->
+      <!-- OLD (WRONG): axis xyz="0 0 1" -->
+      <!-- NEW (CORRECT): axis xyz="0 1 0" -->
+      <!-- -->
+      <!-- Wheels rotate around Y axis in this URDF because -->
+      <!-- cylinder visual is rotated using rpy="${pi/2} 0 0" -->
+      <!-- ================================================= -->
       <axis xyz="0 1 0"/>
-      <!-- Optional dynamics -->
       <dynamics damping="0.01" friction="0.1"/>
     </joint>
   </xacro:macro>
   <!-- ================= WHEELS ================= -->
-  <!-- Four wheels generated using macro -->
   <xacro:wheel name="front_left"  x_sign=" 1" y_sign=" 1"/>
   <xacro:wheel name="front_right" x_sign=" 1" y_sign="-1"/>
@@ -131,9 +125,7 @@
   <xacro:wheel name="rear_right"  x_sign="-1" y_sign="-1"/>
   <!-- ================= IMU ================= -->
-  <!-- Inertial Measurement Unit sensor -->
   <link name="imu_link">
     <visual>
       <geometry>
-        <!-- Small box representing IMU -->
         <box size="0.03 0.03 0.01"/>
       </geometry>
@@ -142,10 +134,14 @@
     <inertial>
       <mass value="0.05"/>
-      <inertia ixx="0.0001" ixy="0" ixz="0"
-               iyy="0.0001" iyz="0"
-               izz="0.0001"/>
+      <inertia
+        ixx="0.0001"
+        ixy="0"
+        ixz="0"
+        iyy="0.0001"
+        iyz="0"
+        izz="0.0001"/>
     </inertial>
   </link>
-  <!-- Fixed IMU on top of base -->
+  <!-- IMU fixed to robot -->
   <joint name="imu_joint" type="fixed">
     <parent link="base_link"/>

Commit message: Add Kinect-based mapping pipeline

File: src/yakizbot_description/urdf/yakizbot.urdf.xacro (robot description, xacro)
@@ -1,40 +1,18 @@
 <?xml version="1.0"?>
-<!--
-  URDF/Xacro model for a 4WD mobile robot (yakizbot)
-  This file defines:
-  - Robot physical dimensions (base + wheels)
-  - Kinematic structure (links & joints)
-  - Inertial properties for simulation/real control
-  - IMU sensor mounting
-  The robot is a 4-wheel drive (4WD) skid-steer platform.
--->
 <robot name="yakizbot" xmlns:xacro="http://www.ros.org/wiki/xacro">
   <!-- ================= PARAMETERS ================= -->
-  <!-- Base dimensions -->
-  <xacro:property name="base_length"   value="0.40"/>
-  <xacro:property name="base_width"    value="0.295"/>
-  <xacro:property name="base_height"   value="0.20"/>
-  <!-- Wheel dimensions -->
-  <xacro:property name="wheel_radius"  value="0.0425"/>
-  <xacro:property name="wheel_width"   value="0.038"/>
-  <!-- Robot geometry -->
-  <xacro:property name="track"         value="0.28"/>
-  <xacro:property name="wheelbase"     value="0.15"/>
+  <xacro:property name="base_length" value="0.40"/>
+  <xacro:property name="base_width" value="0.295"/>
+  <xacro:property name="base_height" value="0.20"/>
+  <xacro:property name="wheel_radius" value="0.0425"/>
+  <xacro:property name="wheel_width" value="0.038"/>
+  <xacro:property name="track" value="0.28"/>
+  <xacro:property name="wheelbase" value="0.15"/>
   <!-- ================= MATERIALS ================= -->
-  <material name="blue">
-    <color rgba="0 0 1 1"/>
-  </material>
-  <material name="black">
-    <color rgba="0 0 0 1"/>
-  </material>
-  <material name="silver">
-    <color rgba="0.79 0.82 0.93 1"/>
-  </material>
-  <material name="dark_grey">
-    <color rgba="0.3 0.3 0.3 1"/>
-  </material>
-  <!-- ================================================= -->
+  <material name="blue"><color rgba="0 0 1 1"/></material>
+  <material name="black"><color rgba="0 0 0 1"/></material>
+  <material name="silver"><color rgba="0.79 0.82 0.93 1"/></material>
+  <!-- ================= BASE ================= -->
   <link name="base_footprint"/>
-  <!-- ================= BASE LINK ================= -->
   <link name="base_link">
     <visual>
@@ -49,99 +27,26 @@
       </geometry>
     </collision>
-    <inertial>
-      <origin xyz="0 0 0.04"/>
-      <mass value="3.0"/>
-      <inertia
-        ixx="0.05"
-        ixy="0.0"
-        ixz="0.0"
-        iyy="0.05"
-        iyz="0.0"
-        izz="0.08"/>
-    </inertial>
   </link>
-  <!-- ================= BASE JOINT ================= -->
   <joint name="base_joint" type="fixed">
     <parent link="base_footprint"/>
     <child link="base_link"/>
-    <!-- Lift robot body above ground -->
     <origin xyz="0 0 ${wheel_radius}" rpy="0 0 0"/>
   </joint>
-  <!-- ================= WHEEL MACRO ================= -->
+  <!-- ================= WHEELS (unchanged logic) ================= -->
   <xacro:macro name="wheel" params="name x_sign y_sign">
-    <!-- Wheel link -->
-    <link name="${name}_wheel">
-      <visual>
-        <geometry>
-          <cylinder radius="${wheel_radius}" length="${wheel_width}"/>
-        </geometry>
-        <!-- Cylinder rotated so wheel looks correct -->
-        <origin rpy="${pi/2} 0 0"/>
-        <material name="blue"/>
-      </visual>
-      <collision>
-        <geometry>
-          <cylinder radius="${wheel_radius}" length="${wheel_width}"/>
-        </geometry>
-        <origin rpy="${pi/2} 0 0"/>
-      </collision>
-      <inertial>
-        <mass value="0.3"/>
-        <inertia
-          ixx="0.001"
-          ixy="0"
-          ixz="0"
-          iyy="0.001"
-          iyz="0"
-          izz="0.001"/>
-      </inertial>
-    </link>
-    <!-- Wheel joint -->
+    <link name="${name}_wheel"/>
     <joint name="${name}_wheel_joint" type="continuous">
       <parent link="base_link"/>
       <child link="${name}_wheel"/>
-      <!-- Wheel position -->
-      <origin
-        xyz="${x_sign * wheelbase/2}
-             ${y_sign * track/2}
-             ${-base_height/2}"
-        rpy="0 0 0"/>
-      <!-- ================================================= -->
-      <!-- FIX: wheel rotation axis -->
-      <!-- OLD (WRONG): axis xyz="0 0 1" -->
-      <!-- NEW (CORRECT): axis xyz="0 1 0" -->
-      <!-- -->
-      <!-- Wheels rotate around Y axis in this URDF because -->
-      <!-- cylinder visual is rotated using rpy="${pi/2} 0 0" -->
-      <!-- ================================================= -->
+      <origin xyz="${x_sign * wheelbase/2} ${y_sign * track/2} ${-base_height/2}" rpy="0 0 0"/>
       <axis xyz="0 1 0"/>
-      <dynamics damping="0.01" friction="0.1"/>
     </joint>
   </xacro:macro>
-  <!-- ================= WHEELS ================= -->
-  <xacro:wheel name="fl"   x_sign=" 1" y_sign=" 1"/>
-  <xacro:wheel name="rl"   x_sign="-1" y_sign=" 1"/>
-  <xacro:wheel name="fr"   x_sign=" 1" y_sign="-1"/>
-  <xacro:wheel name="rr"   x_sign="-1" y_sign="-1"/>
+  <xacro:wheel name="fl" x_sign="1" y_sign="1"/>
+  <xacro:wheel name="rl" x_sign="-1" y_sign="1"/>
+  <xacro:wheel name="fr" x_sign="1" y_sign="-1"/>
+  <xacro:wheel name="rr" x_sign="-1" y_sign="-1"/>
   <!-- ================= IMU ================= -->
-  <link name="imu_link">
-    <visual>
-      <geometry>
-        <box size="0.03 0.03 0.01"/>
-      </geometry>
-      <material name="silver"/>
-    </visual>
-    <inertial>
-      <mass value="0.05"/>
-      <inertia
-        ixx="0.0001"
-        ixy="0"
-        ixz="0"
-        iyy="0.0001"
-        iyz="0"
-        izz="0.0001"/>
-    </inertial>
-  </link>
-  <!-- IMU fixed to robot -->
+  <link name="imu_link"/>
   <joint name="imu_joint" type="fixed">
     <parent link="base_link"/>
@@ -149,3 +54,34 @@
     <origin xyz="0 0 ${base_height/2}" rpy="0 0 0"/>
   </joint>
+  <!-- ================================================= -->
+  <!-- ================= KINECT FIX ================= -->
+  <!-- ================================================= -->
+  <!-- Physical camera body -->
+  <link name="kinect_link">
+    <visual>
+      <geometry>
+        <box size="0.28 0.08 0.07"/>
+      </geometry>
+      <material name="blue"/>
+    </visual>
+    <collision>
+      <geometry>
+        <box size="0.28 0.08 0.07"/>
+      </geometry>
+    </collision>
+  </link>
+  <!-- FIX: only ONE mount transform -->
+  <joint name="kinect_joint" type="fixed">
+    <parent link="base_link"/>
+    <child link="kinect_link"/>
+    <origin xyz="0.15 0 0.25" rpy="0 0 0"/>
+  </joint>
+  <!-- Depth frame (sensor optical frame) -->
+  <link name="kinect_depth"/>
+  <joint name="kinect_depth_joint" type="fixed">
+    <parent link="kinect_link"/>
+    <child link="kinect_depth"/>
+    <!-- FIX: must be identity transform (no offset) -->
+    <origin xyz="0 0 0" rpy="0 0 0"/>
+  </joint>
 </robot>

Commit message: fix kinect setup and update slam toolbox configuration and launch

File: src/yakizbot_description/urdf/yakizbot.urdf.xacro (robot description, xacro)
@@ -9,7 +9,12 @@
   <xacro:property name="track" value="0.28"/>
   <xacro:property name="wheelbase" value="0.15"/>
+  <!-- Kinect 1 real dimensions: 9.8in wide x 3in tall x 3in deep -->
+  <xacro:property name="kinect_w" value="0.249"/>  <!-- 9.8 in → m -->
+  <xacro:property name="kinect_h" value="0.076"/>  <!-- 3.0 in → m -->
+  <xacro:property name="kinect_d" value="0.076"/>  <!-- 3.0 in → m -->
   <!-- ================= MATERIALS ================= -->
+  <material name="black"><color rgba="0 0 0 1"/></material>
   <material name="blue"><color rgba="0 0 1 1"/></material>
-  <material name="black"><color rgba="0 0 0 1"/></material>
+  <material name="green"><color rgba="0 0.8 0 1"/></material>
   <material name="silver"><color rgba="0.79 0.82 0.93 1"/></material>
   <!-- ================= BASE ================= -->
@@ -33,5 +38,5 @@
     <origin xyz="0 0 ${wheel_radius}" rpy="0 0 0"/>
   </joint>
-  <!-- ================= WHEELS (unchanged logic) ================= -->
+  <!-- ================= WHEELS ================= -->
   <xacro:macro name="wheel" params="name x_sign y_sign">
     <link name="${name}_wheel"/>
@@ -55,5 +60,10 @@
   </joint>
   <!-- ================================================= -->
-  <!-- ================= KINECT FIX ================= -->
+  <!-- ================= KINECT (XBOX 360) ================= -->
+  <!--                                                       -->
+  <!--  Mounted centered (Y=0) between FL & FR wheels,       -->
+  <!--  sitting on top of the base_link.                     -->
+  <!--  X=0  →  centred front-to-back                        -->
+  <!--  Z = base_height/2 + kinect_h/2  →  rests on top      -->
   <!-- ================================================= -->
   <!-- Physical camera body -->
@@ -61,27 +71,42 @@
     <visual>
       <geometry>
-        <box size="0.28 0.08 0.07"/>
+        <box size="${kinect_d} ${kinect_w} ${kinect_h}"/>
+        <!-- x=depth, y=width, z=height so the bar lies across the robot -->
       </geometry>
-      <material name="blue"/>
+      <material name="green"/>
     </visual>
     <collision>
       <geometry>
-        <box size="0.28 0.08 0.07"/>
+        <box size="${kinect_d} ${kinect_w} ${kinect_h}"/>
       </geometry>
     </collision>
   </link>
-  <!-- FIX: only ONE mount transform -->
+  <!-- Mount: centered between FL & FR, sitting on top of base -->
   <joint name="kinect_joint" type="fixed">
     <parent link="base_link"/>
     <child link="kinect_link"/>
-    <origin xyz="0.15 0 0.25" rpy="0 0 0"/>
+    <origin xyz="${base_length/4} 0 ${base_height/2 + kinect_h/2}" rpy="0 0 0"/>
   </joint>
-  <!-- Depth frame (sensor optical frame) -->
+  <!-- Sensor origin (depth sensor centre) -->
+  <!-- Kinect 1 depth sensor is slightly left of centre (~2 cm).      -->
+  <!-- Kept at (0,0,0) relative to kinect_link for simplicity;        -->
+  <!-- adjust x/y if you need sub-centimetre accuracy.                -->
   <link name="kinect_depth"/>
   <joint name="kinect_depth_joint" type="fixed">
     <parent link="kinect_link"/>
     <child link="kinect_depth"/>
-    <!-- FIX: must be identity transform (no offset) -->
     <origin xyz="0 0 0" rpy="0 0 0"/>
   </joint>
+  <!-- Optical frame (ROS convention)  -->
+  <!--  Standard ROS camera optical frame:                             -->
+  <!--    Z  points forward  (into the scene)                         -->
+  <!--    Y  points downward                                           -->
+  <!--    X  points right                                              -->
+  <!--  Achieved by rpy = (-π/2, 0, -π/2) from the URDF body frame.  -->
+  <link name="kinect_depth_optical_frame"/>
+  <joint name="kinect_depth_optical_joint" type="fixed">
+    <parent link="kinect_depth"/>
+    <child link="kinect_depth_optical_frame"/>
+    <origin xyz="0 0 0" rpy="${-pi/2} 0 ${-pi/2}"/>
+  </joint>
 </robot>

Commit message: feat: add yakizbot_patrol package for autonomous patrolling

File: src/yakizbot_description/urdf/yakizbot.urdf.xacro (robot description, xacro)
@@ -2,6 +2,6 @@
 <robot name="yakizbot" xmlns:xacro="http://www.ros.org/wiki/xacro">
   <!-- ================= PARAMETERS ================= -->
-  <xacro:property name="base_length" value="0.40"/>
-  <xacro:property name="base_width" value="0.295"/>
+  <xacro:property name="base_length" value="0.295"/>
+  <xacro:property name="base_width" value="0.40"/>
   <xacro:property name="base_height" value="0.20"/>
   <xacro:property name="wheel_radius" value="0.0425"/>
